Commit message: Fix head pitch zero pose, set license to GPL-3.0-only
Servos 19/20 at 120 deg = head level/centred on the real robot, but
the PC-software Offset (-135) tilted the model head up 15 deg at 120.
Add an urdf_offset field to servo_map.yaml (overrides pc_offset for
the URDF) and set head pitch zero to q = servo - 120, giving
limits [-0.26180, 0.61087] rad. Zero pose head_pitch_joint becomes
0.0 in the SRDF; add head_pitch_link <-> l_elbow_link to the
never-colliding table.

Also set <license> to GPL-3.0-only to match the existing LICENSE
file, and document the exception, the joint-limit decision and
third-party mesh provenance in README.

File: urdf/alpha2.urdf (robot description, URDF)
Before this commit: robot alpha2, 29 links, 28 joints
Joints:
- joint head_pitch_joint: limit lower=-0.52360 upper=0.34907 effort=1.5 velocity=5.0 -> lower=-0.26180 upper=0.61087 effort=1.5 velocity=5.0

Commit message: Replace convex-hull collision with CoACD decomposition; add MuJoCo model
Collision geometry: single convex hull per link -> CoACD convex
decomposition (up to 8 pieces per link, 160 total), clamped to the
visual mesh bounding box so sole heights and extents match the
visual. Improves concavity handling in the feet and torso.

SRDF collision-disable table recomputed against the new pieces: 20
adjacent, 2 default-overlapping, 83 never colliding (105 pairs stay
enabled). base_footprint moved to the default-stance ground plane
(0.2206 m).

New MuJoCo physics copy for validation:
- urdf/alpha2_mujoco.urdf: collision pieces only, no visuals/frame links
- mujoco/stand_test.py: free base + ground + position servos, joint
  armature 0.005 and implicitfast integration (both required for
  numerical stability at 8e-7 kg*m^2 principal inertia)

Note: the 21 original single-hull collision STLs are now unreferenced
by any URDF and are left in the tree pending a cleanup decision.

File: urdf/alpha2.urdf (robot description, URDF)
Before this commit: robot alpha2, 29 links, 28 joints
Links:
- link base_link: geometry collision mesh filename=package://alpha2_description/meshes/collision/base_link_0.s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; collision mesh filename=package://alpha2_description/meshes/collision/base_link_1.s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
- link head_pitch_link: geometry collision mesh filename=package://alpha2_description/meshes/collision/head_pitch_li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; collision mesh filename=package://alpha2_description/meshes/collision/head_pitch_li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
- link l_ankle_pitch_link: geometry collision mesh filename=package://alpha2_description/meshes/collision/l_ankle_pitch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; collision mesh filename=package://alpha2_description/meshes/collision/l_ankle_pitch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
- link l_ankle_roll_link: geometry collision mesh filename=package://alpha2_description/meshes/collision/l_ankle_roll_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; collision mesh filename=package://alpha2_description/meshes/collision/l_ankle_roll_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
- link l_elbow_link: geometry collision mesh filename=package://alpha2_description/meshes/collision/l_elbow_link_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; collision mesh filename=package://alpha2_description/meshes/collision/l_elbow_link_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
- link l_hand_link: geometry collision mesh filename=package://alpha2_description/meshes/collision/l_hand_link_0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; collision mesh filename=package://alpha2_description/meshes/collision/l_hand_link_1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
- link l_hip_pitch_link: geometry collision mesh filename=package://alpha2_description/meshes/collision/l_hip_pitch_l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; collision mesh filename=package://alpha2_description/meshes/collision/l_hip_pitch_l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
- link l_hip_roll_link: geometry collision mesh filename=package://alpha2_description/meshes/collision/l_hip_roll_li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; collision mesh filename=package://alpha2_description/meshes/collision/l_hip_roll_li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
- link l_knee_link: geometry collision mesh filename=package://alpha2_description/meshes/collision/l_knee_link_0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; collision mesh filename=package://alpha2_description/meshes/collision/l_knee_link_1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
- link l_shoulder_pitch_link: geometry collision mesh filename=package://alpha2_description/meshes/collision/l_shoulder_pi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; collision mesh filename=package://alpha2_description/meshes/collision/l_shoulder_pi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
- link l_shoulder_roll_link: geometry collision mesh filename=package://alpha2_description/meshes/collision/l_shoulder_ro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; collision mesh filename=package://alpha2_description/meshes/collision/l_shoulder_ro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
- link r_ankle_pitch_link: geometry collision mesh filename=package://alpha2_description/meshes/collision/r_ankle_pitch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; collision mesh filename=package://alpha2_description/meshes/collision/r_ankle_pitch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
- link r_ankle_roll_link: geometry collision mesh filename=package://alpha2_description/meshes/collision/r_ankle_roll_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; collision mesh filename=package://alpha2_description/meshes/collision/r_ankle_roll_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
- link r_elbow_link: geometry collision mesh filename=package://alpha2_description/meshes/collision/r_elbow_link_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; collision mesh filename=package://alpha2_description/meshes/collision/r_elbow_link_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
- link r_hand_link: geometry collision mesh filename=package://alpha2_description/meshes/collision/r_hand_link_0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; collision mesh filename=package://alpha2_description/meshes/collision/r_hand_link_1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
- link r_hip_pitch_link: geometry collision mesh filename=package://alpha2_description/meshes/collision/r_hip_pitch_l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; collision mesh filename=package://alpha2_description/meshes/collision/r_hip_pitch_l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
- link r_hip_roll_link: geometry collision mesh filename=package://alpha2_description/meshes/collision/r_hip_roll_li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; collision mesh filename=package://alpha2_description/meshes/collision/r_hip_roll_li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
- link r_knee_link: geometry collision mesh filename=package://alpha2_description/meshes/collision/r_knee_link_0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; collision mesh filename=package://alpha2_description/meshes/collision/r_knee_link_1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
- link r_shoulder_pitch_link: geometry collision mesh filename=package://alpha2_description/meshes/collision/r_shoulder_pi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; collision mesh filename=package://alpha2_description/meshes/collision/r_shoulder_pi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
- link r_shoulder_roll_link: geometry collision mesh filename=package://alpha2_description/meshes/collision/r_shoulder_ro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; collision mesh filename=package://alpha2_description/meshes/collision/r_shoulder_ro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
Joints:
- joint base_footprint_joint: origin xyz=0 0 0.218642 rpy=0 0 0 -> xyz=0 0 0.220606 rpy=0 0 0
- joint l_hand_tip_joint: origin xyz=0.021756 -0.011977 -0.038685 rpy=0 0 0 -> xyz=0.021396 -0.012449 -0.038527 rpy=0 0 0
- joint l_sole_frame_joint: origin xyz=0.000202 0.009880 -0.027222 rpy=0 0 0 -> xyz=0.000213 0.016948 -0.027969 rpy=0 0 0
- joint r_hand_tip_joint: origin xyz=0.000475 0.011671 -0.038763 rpy=0 0 0 -> xyz=-0.000000 0.012449 -0.038605 rpy=0 0 0
- joint r_sole_frame_joint: origin xyz=0.005153 -0.014847 -0.027969 rpy=0 0 0 -> xyz=0.000213 -0.016948 -0.027969 rpy=0 0 0

Commit message: Add per-servo mass/torque data and Isaac Sim import path
Replace the flat effort=1.5 N*m placeholder with real per-servo stall
torque from the UBTECH servo table: 12 kg*cm (1.1768 N*m) for the
light servos (IDs 2,3,5,6,17-20, 40.3 g) and 20 kg*cm (1.9613 N*m)
for the heavy ones (IDs 1,4,7-16, 52.8 g). Joint inertia and link
masses updated to match the corrected per-servo mass split; total
mass still sums to exactly 2.300 kg. Adds servo_mass_g / torque_kgcm
/ torque_nm to servo_map.yaml so the physics scripts read the real
numbers instead of a constant.

- mujoco/stand_test.py: per-servo forcerange from servo_map.yaml;
  README records that 45/202 official actions still saturate a
  servo under the real torque limits (hip rolls mainly), p90 joint
  tracking error 11.5 deg.
- urdf/alpha2_isaac.urdf: alpha2.urdf with relative mesh paths for
  the Isaac Sim importer (all 181 mesh refs verified to resolve).
- isaac/import_and_stand.py + isaac/README.md: Isaac 4.x import and
  5 s standing test. NOT run (no GPU/NVIDIA package index available);
  offline pre-flight checks only. Drive gains converted N*m/rad ->
  N*m/deg because USD angular drives are per degree.

File: urdf/alpha2.urdf (robot description, URDF)
Before this commit: robot alpha2, 29 links, 28 joints
Links:
- link base_link: mass 0.42377 -> 0.41816
- link head_pitch_link: mass 0.26548 -> 0.26086
- link head_yaw_link: mass 0.05123 -> 0.05101
- link l_ankle_pitch_link: mass 0.08919 -> 0.08844
- link l_ankle_roll_link: mass 0.14066 -> 0.13886
- link l_elbow_link: mass 0.09679 -> 0.09563
- link l_hand_link: mass 0.04764 -> 0.04749
- link l_hip_pitch_link: mass 0.09681 -> 0.09591
- link l_hip_roll_link: mass 0.07747 -> 0.07696
- link l_knee_link: mass 0.10587 -> 0.10478
- link l_shoulder_pitch_link: mass 0.05261 -> 0.06486
- link l_shoulder_roll_link: mass 0.07270 -> 0.07204
- link r_ankle_pitch_link: mass 0.08919 -> 0.08844
- link r_ankle_roll_link: mass 0.14069 -> 0.13889
- link r_elbow_link: mass 0.09679 -> 0.09563
- link r_hand_link: mass 0.04764 -> 0.04749
- link r_hip_pitch_link: mass 0.09681 -> 0.09591
- link r_hip_roll_link: mass 0.07747 -> 0.07696
- link r_knee_link: mass 0.10587 -> 0.10478
- link r_shoulder_pitch_link: mass 0.05261 -> 0.06486
- link r_shoulder_roll_link: mass 0.07270 -> 0.07204
Joints:
- joint head_pitch_joint: limit lower=-0.26180 upper=0.61087 effort=1.5 velocity=5.0 -> lower=-0.26180 upper=0.61087 effort=1.1768 velocity=5.0
- joint head_yaw_joint: limit lower=-0.78540 upper=0.78540 effort=1.5 velocity=5.0 -> lower=-0.78540 upper=0.78540 effort=1.1768 velocity=5.0
- joint l_ankle_pitch_joint: limit lower=-1.30900 upper=1.83260 effort=1.5 velocity=5.0 -> lower=-1.30900 upper=1.83260 effort=1.9613 velocity=5.0
- joint l_ankle_roll_joint: limit lower=-1.22173 upper=0.34907 effort=1.5 velocity=5.0 -> lower=-1.22173 upper=0.34907 effort=1.9613 velocity=5.0
- joint l_elbow_joint: limit lower=-1.39626 upper=0.87266 effort=1.5 velocity=5.0 -> lower=-1.39626 upper=0.87266 effort=1.1768 velocity=5.0
- joint l_hand_joint: limit lower=-0.43633 upper=0.08727 effort=1.5 velocity=5.0 -> lower=-0.43633 upper=0.08727 effort=1.1768 velocity=5.0
- joint l_hip_pitch_joint: limit lower=-2.53073 upper=0.95993 effort=1.5 velocity=5.0 -> lower=-2.53073 upper=0.95993 effort=1.9613 velocity=5.0
- joint l_hip_roll_joint: limit lower=-1.43117 upper=0.31416 effort=1.5 velocity=5.0 -> lower=-1.43117 upper=0.31416 effort=1.9613 velocity=5.0
- joint l_knee_joint: limit lower=-1.39626 upper=2.00713 effort=1.5 velocity=5.0 -> lower=-1.39626 upper=2.00713 effort=1.9613 velocity=5.0
- joint l_shoulder_pitch_joint: limit lower=-1.83260 upper=2.18166 effort=1.5 velocity=5.0 -> lower=-1.83260 upper=2.18166 effort=1.9613 velocity=5.0
- joint l_shoulder_roll_joint: limit lower=0.00000 upper=2.79253 effort=1.5 velocity=5.0 -> lower=0.00000 upper=2.79253 effort=1.1768 velocity=5.0
- joint r_ankle_pitch_joint: limit lower=-1.83260 upper=1.30900 effort=1.5 velocity=5.0 -> lower=-1.83260 upper=1.30900 effort=1.9613 velocity=5.0
- joint r_ankle_roll_joint: limit lower=-0.34907 upper=1.22173 effort=1.5 velocity=5.0 -> lower=-0.34907 upper=1.22173 effort=1.9613 velocity=5.0
- joint r_elbow_joint: limit lower=-1.04720 upper=1.22173 effort=1.5 velocity=5.0 -> lower=-1.04720 upper=1.22173 effort=1.1768 velocity=5.0
- joint r_hand_joint: limit lower=-0.43633 upper=0.08727 effort=1.5 velocity=5.0 -> lower=-0.43633 upper=0.08727 effort=1.1768 velocity=5.0
- joint r_hip_pitch_joint: limit lower=-0.95993 upper=2.53073 effort=1.5 velocity=5.0 -> lower=-0.95993 upper=2.53073 effort=1.9613 velocity=5.0
- joint r_hip_roll_joint: limit lower=-0.34907 upper=1.39626 effort=1.5 velocity=5.0 -> lower=-0.34907 upper=1.39626 effort=1.9613 velocity=5.0
- joint r_knee_joint: limit lower=-2.00713 upper=1.39626 effort=1.5 velocity=5.0 -> lower=-2.00713 upper=1.39626 effort=1.9613 velocity=5.0
- joint r_shoulder_pitch_joint: limit lower=-2.18166 upper=1.83260 effort=1.5 velocity=5.0 -> lower=-2.18166 upper=1.83260 effort=1.9613 velocity=5.0
- joint r_shoulder_roll_joint: limit lower=-2.79253 upper=0.00000 effort=1.5 velocity=5.0 -> lower=-2.79253 upper=0.00000 effort=1.1768 velocity=5.0

File: urdf/alpha2_mujoco.urdf (robot description, URDF)
Before this commit: robot alpha2, 21 links, 20 joints
Links:
- link base_link: mass 0.42377 -> 0.41816
- link head_pitch_link: mass 0.26548 -> 0.26086
- link head_yaw_link: mass 0.05123 -> 0.05101
- link l_ankle_pitch_link: mass 0.08919 -> 0.08844
- link l_ankle_roll_link: mass 0.14066 -> 0.13886
- link l_elbow_link: mass 0.09679 -> 0.09563
- link l_hand_link: mass 0.04764 -> 0.04749
- link l_hip_pitch_link: mass 0.09681 -> 0.09591
- link l_hip_roll_link: mass 0.07747 -> 0.07696
- link l_knee_link: mass 0.10587 -> 0.10478
- link l_shoulder_pitch_link: mass 0.05261 -> 0.06486
- link l_shoulder_roll_link: mass 0.07270 -> 0.07204
- link r_ankle_pitch_link: mass 0.08919 -> 0.08844
- link r_ankle_roll_link: mass 0.14069 -> 0.13889
- link r_elbow_link: mass 0.09679 -> 0.09563
- link r_hand_link: mass 0.04764 -> 0.04749
- link r_hip_pitch_link: mass 0.09681 -> 0.09591
- link r_hip_roll_link: mass 0.07747 -> 0.07696
- link r_knee_link: mass 0.10587 -> 0.10478
- link r_shoulder_pitch_link: mass 0.05261 -> 0.06486
- link r_shoulder_roll_link: mass 0.07270 -> 0.07204
Joints:
- joint head_pitch_joint: limit lower=-0.26180 upper=0.61087 effort=1.5 velocity=5.0 -> lower=-0.26180 upper=0.61087 effort=1.1768 velocity=5.0
- joint head_yaw_joint: limit lower=-0.78540 upper=0.78540 effort=1.5 velocity=5.0 -> lower=-0.78540 upper=0.78540 effort=1.1768 velocity=5.0
- joint l_ankle_pitch_joint: limit lower=-1.30900 upper=1.83260 effort=1.5 velocity=5.0 -> lower=-1.30900 upper=1.83260 effort=1.9613 velocity=5.0
- joint l_ankle_roll_joint: limit lower=-1.22173 upper=0.34907 effort=1.5 velocity=5.0 -> lower=-1.22173 upper=0.34907 effort=1.9613 velocity=5.0
- joint l_elbow_joint: limit lower=-1.39626 upper=0.87266 effort=1.5 velocity=5.0 -> lower=-1.39626 upper=0.87266 effort=1.1768 velocity=5.0
- joint l_hand_joint: limit lower=-0.43633 upper=0.08727 effort=1.5 velocity=5.0 -> lower=-0.43633 upper=0.08727 effort=1.1768 velocity=5.0
- joint l_hip_pitch_joint: limit lower=-2.53073 upper=0.95993 effort=1.5 velocity=5.0 -> lower=-2.53073 upper=0.95993 effort=1.9613 velocity=5.0
- joint l_hip_roll_joint: limit lower=-1.43117 upper=0.31416 effort=1.5 velocity=5.0 -> lower=-1.43117 upper=0.31416 effort=1.9613 velocity=5.0
- joint l_knee_joint: limit lower=-1.39626 upper=2.00713 effort=1.5 velocity=5.0 -> lower=-1.39626 upper=2.00713 effort=1.9613 velocity=5.0
- joint l_shoulder_pitch_joint: limit lower=-1.83260 upper=2.18166 effort=1.5 velocity=5.0 -> lower=-1.83260 upper=2.18166 effort=1.9613 velocity=5.0
- joint l_shoulder_roll_joint: limit lower=0.00000 upper=2.79253 effort=1.5 velocity=5.0 -> lower=0.00000 upper=2.79253 effort=1.1768 velocity=5.0
- joint r_ankle_pitch_joint: limit lower=-1.83260 upper=1.30900 effort=1.5 velocity=5.0 -> lower=-1.83260 upper=1.30900 effort=1.9613 velocity=5.0
- joint r_ankle_roll_joint: limit lower=-0.34907 upper=1.22173 effort=1.5 velocity=5.0 -> lower=-0.34907 upper=1.22173 effort=1.9613 velocity=5.0
- joint r_elbow_joint: limit lower=-1.04720 upper=1.22173 effort=1.5 velocity=5.0 -> lower=-1.04720 upper=1.22173 effort=1.1768 velocity=5.0
- joint r_hand_joint: limit lower=-0.43633 upper=0.08727 effort=1.5 velocity=5.0 -> lower=-0.43633 upper=0.08727 effort=1.1768 velocity=5.0
- joint r_hip_pitch_joint: limit lower=-0.95993 upper=2.53073 effort=1.5 velocity=5.0 -> lower=-0.95993 upper=2.53073 effort=1.9613 velocity=5.0
- joint r_hip_roll_joint: limit lower=-0.34907 upper=1.39626 effort=1.5 velocity=5.0 -> lower=-0.34907 upper=1.39626 effort=1.9613 velocity=5.0
- joint r_knee_joint: limit lower=-2.00713 upper=1.39626 effort=1.5 velocity=5.0 -> lower=-2.00713 upper=1.39626 effort=1.9613 velocity=5.0
- joint r_shoulder_pitch_joint: limit lower=-2.18166 upper=1.83260 effort=1.5 velocity=5.0 -> lower=-2.18166 upper=1.83260 effort=1.9613 velocity=5.0
- joint r_shoulder_roll_joint: limit lower=-2.79253 upper=0.00000 effort=1.5 velocity=5.0 -> lower=-2.79253 upper=0.00000 effort=1.1768 velocity=5.0

Commit message: Add Gazebo Sim (Harmonic) support
- model.sdf + model.config: generated from urdf/alpha2.urdf with
  libsdformat 14 (SDF 1.11), mesh URIs model://alpha2_description/...
- gazebo/alpha2_world.sdf: DART 1 ms, ground plane, model via <include>,
  20 JointPositionController plugins (kp 20, kv 0.5) whose torque limits
  are read from config/servo_map.yaml per servo (1.1768 / 1.9613 N*m)

URDF changes for Gazebo: camera_link and accel_link get a negligible
10 mg inertial plus <preserveFixedJoint> so sdformat keeps them as
sensor mounts instead of dropping massless links; foot friction
mu1/mu2 = 1.0 on both ankle_roll links. The <gazebo> tags are ignored
by ROS/RViz/MoveIt.

Verified offline (NOT simulated - no Gazebo runtime/GPU here):
model.sdf parses, 181 mesh URIs resolve, all 20 controller torque
limits match servo_map.yaml, urdf/alpha2.urdf still parses with 29
links / 20 revolute / 160 collisions and total mass 2.30002 kg
(2.300 + 2 x 10 mg).

Also note in README/servo_map.yaml that effort is the servo STALL
torque (maintainer-confirmed) and that no torque-speed curve is
modelled, so available torque while moving is lower.

File: urdf/alpha2.urdf (robot description, URDF)
Before this commit: robot alpha2, 29 links, 28 joints
Links:
- link accel_link: mass None -> 1e-05
- link camera_link: mass None -> 1e-05

Commit message: Correct light-servo stall torque to 8 kg*cm; add servo travel envelope
Resolves the manual-vs-model discrepancy flagged in the previous
commit: the Alpha 2 manual lists 8 kg*cm for the light servos, so the
light servos (IDs 2,3,5,6,17-20) drop from 12 kg*cm / 1.1768 N*m to
8 kg*cm / 0.7845 N*m. Heavy servos (IDs 1,4,7-16) unchanged at
20 kg*cm / 1.9613 N*m.

Propagated to every consumer of the torque value:
- config/servo_map.yaml: torque_kgcm / torque_nm for 10 servos
- urdf/alpha2.urdf + urdf/alpha2_mujoco.urdf: effort on 10 joints
- model.sdf + gazebo/alpha2_world.sdf: cmd_max/cmd_min on 10
  controllers
Verified all 20 URDF efforts and all 20 Gazebo cmd_max values match
servo_map.yaml exactly; mass still 2.30002 kg; 181 mesh URIs resolve.

New config/servo_envelope.yaml: per-servo union of the measured
SERVO_CALIBRATION range and the range the 202 official actions
actually command, with frames_outside_calibration counts. NOT used by
the URDF - the measured limits are deliberately kept - it is there so
the official actions can be simulated without clipping.

README: records the maintainer's ground truth that on the real robot
every official action except FrontStand and stretch forward runs
without falling, the identified cause of the 'body being hollowed
out' fall (commanded values outside the calibrated range, so the deep
squat is unreachable and the model tips onto its toes), that Sirius
needs smooth interpolation rather than move-then-hold, and the
best-fit setting (smooth interpolation + 15 deg wider ranges) which
matches the real robot for 199 of 202 actions. Notes the remaining
london-bridge discrepancy is unexplained, and that the COM/ZMP-margin
statistic was not reliable enough to use as evidence.

File: urdf/alpha2.urdf (robot description, URDF)
Before this commit: robot alpha2, 29 links, 28 joints
Joints:
- joint head_pitch_joint: limit lower=-0.26180 upper=0.61087 effort=1.1768 velocity=5.0 -> lower=-0.26180 upper=0.61087 effort=0.7845 velocity=5.0
- joint head_yaw_joint: limit lower=-0.78540 upper=0.78540 effort=1.1768 velocity=5.0 -> lower=-0.78540 upper=0.78540 effort=0.7845 velocity=5.0
- joint l_elbow_joint: limit lower=-1.39626 upper=0.87266 effort=1.1768 velocity=5.0 -> lower=-1.39626 upper=0.87266 effort=0.7845 velocity=5.0
- joint l_hand_joint: limit lower=-0.43633 upper=0.08727 effort=1.1768 velocity=5.0 -> lower=-0.43633 upper=0.08727 effort=0.7845 velocity=5.0
- joint l_shoulder_roll_joint: limit lower=0.00000 upper=2.79253 effort=1.1768 velocity=5.0 -> lower=0.00000 upper=2.79253 effort=0.7845 velocity=5.0
- joint r_elbow_joint: limit lower=-1.04720 upper=1.22173 effort=1.1768 velocity=5.0 -> lower=-1.04720 upper=1.22173 effort=0.7845 velocity=5.0
- joint r_hand_joint: limit lower=-0.43633 upper=0.08727 effort=1.1768 velocity=5.0 -> lower=-0.43633 upper=0.08727 effort=0.7845 velocity=5.0
- joint r_shoulder_roll_joint: limit lower=-2.79253 upper=0.00000 effort=1.1768 velocity=5.0 -> lower=-2.79253 upper=0.00000 effort=0.7845 velocity=5.0

File: urdf/alpha2_mujoco.urdf (robot description, URDF)
Before this commit: robot alpha2, 21 links, 20 joints
Joints:
- joint head_pitch_joint: limit lower=-0.26180 upper=0.61087 effort=1.1768 velocity=5.0 -> lower=-0.26180 upper=0.61087 effort=0.7845 velocity=5.0
- joint head_yaw_joint: limit lower=-0.78540 upper=0.78540 effort=1.1768 velocity=5.0 -> lower=-0.78540 upper=0.78540 effort=0.7845 velocity=5.0
- joint l_elbow_joint: limit lower=-1.39626 upper=0.87266 effort=1.1768 velocity=5.0 -> lower=-1.39626 upper=0.87266 effort=0.7845 velocity=5.0
- joint l_hand_joint: limit lower=-0.43633 upper=0.08727 effort=1.1768 velocity=5.0 -> lower=-0.43633 upper=0.08727 effort=0.7845 velocity=5.0
- joint l_shoulder_roll_joint: limit lower=0.00000 upper=2.79253 effort=1.1768 velocity=5.0 -> lower=0.00000 upper=2.79253 effort=0.7845 velocity=5.0
- joint r_elbow_joint: limit lower=-1.04720 upper=1.22173 effort=1.1768 velocity=5.0 -> lower=-1.04720 upper=1.22173 effort=0.7845 velocity=5.0
- joint r_hand_joint: limit lower=-0.43633 upper=0.08727 effort=1.1768 velocity=5.0 -> lower=-0.43633 upper=0.08727 effort=0.7845 velocity=5.0
- joint r_shoulder_roll_joint: limit lower=-2.79253 upper=0.00000 effort=1.1768 velocity=5.0 -> lower=-2.79253 upper=0.00000 effort=0.7845 velocity=5.0
